Commit message: O robo está andando, havia um erro no calculo do dt

File: ros2_ws/src/odom_pkg/urdf/diff_bot.urdf (robot description, URDF)
Before this commit: robot diff_bot, 5 links, 4 joints
Links:
- link caster_wheel: mass 0.2 -> 0.1; geometry collision sphere radius=0.025; visual sphere radius=0.025
- link chassis: mass 5.0 -> 2.0; geometry collision box size=0.30 0.16 0.08; visual box size=0.30 0.16 0.08
- link left_wheel: mass 0.5 -> 0.2; geometry collision cylinder length=0.03 radius=0.05; visual cylinder length=0.03 radius=0.05
- link right_wheel: mass 0.5 -> 0.2; geometry collision cylinder length=0.03 radius=0.05; visual cylinder length=0.03 radius=0.05
Joints:
- joint caster_joint: origin xyz=0.15 0 -0.05 -> xyz=0.10 0 -0.025
- joint chassis_joint: origin xyz=0 0 0.1 -> xyz=0 0 0.05
- joint left_wheel_joint: origin xyz=-0.1 0.175 0 rpy=-1.5707 0 0 -> xyz=-0.05 0.11 0 rpy=-1.5707 0 0
- joint right_wheel_joint: origin xyz=-0.1 -0.175 0 rpy=-1.5707 0 0 -> xyz=-0.05 -0.11 0 rpy=-1.5707 0 0
